File: OpenBMS.sch (KiCad schematic (older format))
At the start: 4 parts

Commit message: removing Stanadard_Interface.pro via CLI
Parts:
- removed MK1, MK2, MK3, MK4: Mounting_Hole_PAD, Mounting_Holes:MountingHole_2.7mm, symbol OpenBMS-rescue:Mounting_Hole_PAD-Mechanical
Connections:
- no-connect marks 4 -> 0
Changed lines of the file:
@@
 Comment4 ""
 $EndDescr
-$Comp
-L OpenBMS-rescue:Mounting_Hole_PAD-Mechanical MK1
-U 1 1 5A6CFED2
-P 650 6700
-F 0 "MK1" H 750 6751 50  0000 L CNN
-F 1 "Mounting_Hole_PAD" H 750 6660 50  0000 L CNN
-F 2 "Mounting_Holes:MountingHole_2.7mm" H 650 6700 50  0001 C CNN
-F 3 "" H 650 6700 50  0001 C CNN
-	1    650  6700
-	1    0    0    -1
-$EndComp
-$Comp
-L OpenBMS-rescue:Mounting_Hole_PAD-Mechanical MK2
-U 1 1 5A6CFF98
-P 650 7000
-F 0 "MK2" H 750 7051 50  0000 L CNN
-F 1 "Mounting_Hole_PAD" H 750 6960 50  0000 L CNN
-F 2 "Mounting_Holes:MountingHole_2.7mm" H 650 7000 50  0001 C CNN
-F 3 "" H 650 7000 50  0001 C CNN
-	1    650  7000
-	1    0    0    -1
-$EndComp
-$Comp
-L OpenBMS-rescue:Mounting_Hole_PAD-Mechanical MK3
-U 1 1 5A6CFFFA
-P 650 7300
-F 0 "MK3" H 750 7351 50  0000 L CNN
-F 1 "Mounting_Hole_PAD" H 750 7260 50  0000 L CNN
-F 2 "Mounting_Holes:MountingHole_2.7mm" H 650 7300 50  0001 C CNN
-F 3 "" H 650 7300 50  0001 C CNN
-	1    650  7300
-	1    0    0    -1
-$EndComp
-$Comp
-L OpenBMS-rescue:Mounting_Hole_PAD-Mechanical MK4
-U 1 1 5A6D003F
-P 650 7600
-F 0 "MK4" H 750 7651 50  0000 L CNN
-F 1 "Mounting_Hole_PAD" H 750 7560 50  0000 L CNN
-F 2 "Mounting_Holes:MountingHole_2.7mm" H 650 7600 50  0001 C CNN
-F 3 "" H 650 7600 50  0001 C CNN
-	1    650  7600
-	1    0    0    -1
-$EndComp
-NoConn ~ 650  6800
-NoConn ~ 650  7100
-NoConn ~ 650  7400
-NoConn ~ 650  7700
 $Sheet
-S 5400 3150 1250 1650
+S 6250 2950 2200 1650
 U 5D167BBA
 F0 "12_Cell_Monitor" 50
@@
 $EndSheet
 $Sheet
-S 2900 3200 1450 1650
+S 4250 2950 1450 1650
 U 5D567F1B
 F0 "Sheet5D567F1A" 50
