File: OpenBMS.sch (KiCad schematic (older format))
At the start: 0 parts

Commit message: Adding everything again - via CLI
Changed lines of the file:
@@
 $Descr A4 11693 8268
 encoding utf-8
-Sheet 1 16
+Sheet 1 17
 Title ""
 Date ""
@@
 $EndDescr
 $Sheet
-S 5850 3000 2200 1650
+S 3500 3100 2200 1650
 U 5D167BBA
 F0 "12_Cell_Monitor" 50
@@
 $EndSheet
 $Sheet
-S 3500 3000 2200 1650
+S 5850 3100 2200 1650
 U 5D567F1B
 F0 "Isolated Communications Interface" 50
 F1 "Standalone_Shield/Standalone_Com_Shield.sch" 50
 $EndSheet
+$Sheet
+S 1600 3100 1750 1650
+U 5D80A62B
+F0 "Molex to Cell Interface" 50
+F1 "LTC6811_12cell_DCARD/Molex_MicroFit_12cell.sch" 50
+$EndSheet
 $EndSCHEMATC
