File: Standalone_Com_Shield.kicad_pcb (KiCad board)
At the start: 2 copper layers, 64.8 x 71.1 mm, 51 parts, among them J1001 Linduino_Test, J1002 Com_H, J1003 Com_L, J1004 Temp6, J1005 Temp5, J1006 Temp4, J1007 Temp3, J1008 Temp2, J1009 Temp1, Q1001 NSV1C201MZ4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

Commit message: added Open Hardware Logo to Standalone_Com_Shield.kicad_pcb via CLI
Parts:
- added REF**: OSHW-Logo2_7.3x6mm_SilkScreen, Symbol:OSHW-Logo2_7.3x6mm_SilkScreen, B.Cu at (166.4, 116.8)
