File: LTC6811_12cell_DCARD/LTC6811_12cell_DCARD.kicad_pcb (KiCad board)
At the start: 2 copper layers, 64.8 x 63.5 mm, 159 parts, among them IC201 LTC6811-1, J102 Cells_1-12, Q1001 BSS308PE, Q1101 BSS308PE, Q1201 BSS308PE, Q1301 BSS308PE, Q1401 BSS308PE, Q301 BSS308PE, Q401 BSS308PE, Q501 BSS308PE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

Commit message: Adding everything again - via CLI
Parts:
- J102: footprint Connector_Molex:Molex_Micro-Fit_3.0_43045-1400_2x07_P3.00mm_Horizontal -> Connector_PinHeader_2.54mm:PinHeader_2x07_P2.54mm_Horizontal
- moved FB201 4.83 mm to (114.9, 112.1)
- moved J102 2.29 mm to (116.2, 108.6), turned to 180 degrees
Connections:
- J102 pad 10: /C4_in -> /C8_in
- J102 pad 11: /C6_in -> /C9_in
- J102 pad 12: /C8_in -> /C10_in
- J102 pad 13: /C10_in -> /C11_in
- J102 pad 2: /C1_in -> /C0_in
- J102 pad 3: /C3_in -> /C1_in
- J102 pad 4: /C5_in -> /C2_in
- J102 pad 5: /C7_in -> /C3_in
- J102 pad 6: /C9_in -> /C4_in
- J102 pad 7: /C11_in -> /C5_in
- J102 pad 8: /C0_in -> /C6_in
- J102 pad 9: /C2_in -> /C7_in
Routing:
- net /C2_in: track 44.6 -> 62.4 mm
- net /C4_in: track 33.1 -> 48.9 mm
- net /C6_in: track 27.6 -> 42.4 mm
- net /C8_in: track 34.3 -> 48.3 mm
- net /C10_in: track 47.0 -> 60.5 mm
- net /C12_in: track 28.2 -> 40.2 mm
- net /C11_in: track 55.4 -> 60.9 mm
- net /C1_in: track 58.4 -> 63.3 mm
- net /C7_in: track 35.5 -> 37.8 mm
- net /C3_in: track 46.9 -> 48.2 mm
- net /C5_in: track 38.0 -> 36.8 mm
- net /C9_in: track 46.9 -> 47.8 mm
- net /C0_in: track 72.4 -> 73.2 mm
