File: LTC6811_12cell_DCARD/LTC6811_12cell_DCARD.sch (KiCad schematic (older format))
At the start: 14 parts, among them IC201 LTC6811-1, J102 Cells_1-12

Commit message: Adding everything again - via CLI
Parts:
- J102: footprint Connector_Molex:Molex_Micro-Fit_3.0_43045-1400_2x07_P3.00mm_Horizontal -> Connector_PinHeader_2.54mm:PinHeader_2x07_P2.54mm_Horizontal; symbol Connector_Generic:Conn_02x07_Top_Bottom -> Connector_Generic:Conn_02x07_Odd_Even
Connections:
- net C0_in: now also J102.2 (Pin_2); no longer J102.8 (Pin_8)
- net C10_in: now also J102.12 (Pin_12); no longer J102.13 (Pin_13)
- net C11_in: now also J102.13 (Pin_13); no longer J102.7 (Pin_7)
- net C1_in: now also J102.3 (Pin_3); no longer J102.2 (Pin_2)
- net C2_in: now also J102.4 (Pin_4); no longer J102.9 (Pin_9)
- net C3_in: now also J102.5 (Pin_5); no longer J102.3 (Pin_3)
- net C4_in: now also J102.6 (Pin_6); no longer J102.10 (Pin_10)
- net C5_in: now also J102.7 (Pin_7); no longer J102.4 (Pin_4)
- net C6_in: now also J102.8 (Pin_8); no longer J102.11 (Pin_11)
- net C7_in: now also J102.9 (Pin_9); no longer J102.5 (Pin_5)
- net C8_in: now also J102.10 (Pin_10); no longer J102.12 (Pin_12)
- net C9_in: now also J102.11 (Pin_11); no longer J102.6 (Pin_6)
Changed lines of the file:
@@
 EESchema Schematic File Version 4
-LIBS:LTC6811_12cell_DCARD-cache
+LIBS:OpenBMS-cache
 EELAYER 30 0
 EELAYER END
 $Descr A 11000 8500
 encoding utf-8
-Sheet 1 14
+Sheet 2 17
 Title ""
 Date ""
@@
 C11
 $Comp
-L Connector_Generic:Conn_02x07_Top_Bottom J102
+L Connector_Generic:Conn_02x07_Odd_Even J102
 U 1 1 5D5581EE
 P 1400 3550
@@
 AR Path="/5D1664F1/5D5581EE" Ref="J?"  Part="1"
 AR Path="/5D167BBA/5D5581EE" Ref="J202"  Part="1"
-F 0 "J102" H 1450 3150 50  0000 C CNN
+F 0 "J202" H 1450 3150 50  0000 C CNN
 F 1 "Cells_1-12" V 1450 3550 50  0000 C CNN
-F 2 "Connector_Molex:Molex_Micro-Fit_3.0_43045-1400_2x07_P3.00mm_Horizontal" H 1400 3550 50  0001 C CNN
+F 2 "Connector_PinHeader_2.54mm:PinHeader_2x07_P2.54mm_Horizontal" H 1400 3550 50  0001 C CNN
 F 3 "~" H 1400 3550 50  0001 C CNN
 	1    1400 3550
@@
 AR Path="/5D1664F1/5D55820F" Ref="R?"  Part="1"
 AR Path="/5D55820F" Ref="R101"  Part="1"
-F 0 "R101" H 2800 6050 50  0000 L CNN
+F 0 "R201" H 2800 6050 50  0000 L CNN
 F 1 "100" V 2750 6050 50  0000 C CNN
 F 2 "Resistor_SMD:R_0805_2012Metric" V 2680 6050 50  0001 C CNN
@@
 AR Path="/5D4F34CB/5D586612" Ref="C?"  Part="1"
 AR Path="/5D167BBA/5D586612" Ref="C202"  Part="1"
-F 0 "C102" H 7665 1196 50  0000 L CNN
+F 0 "C202" H 7665 1196 50  0000 L CNN
 F 1 "1u" H 7665 1105 50  0000 L CNN
 F 2 "Capacitor_SMD:C_0805_2012Metric" H 7588 1000 50  0001 C CNN
@@
 AR Path="/5D4F34CB/5D586622" Ref="C?"  Part="1"
 AR Path="/5D167BBA/5D586622" Ref="C201"  Part="1"
-F 0 "C101" H 5515 2046 50  0000 L CNN
+F 0 "C201" H 5515 2046 50  0000 L CNN
 F 1 "1u" H 5515 1955 50  0000 L CNN
 F 2 "Capacitor_SMD:C_0805_2012Metric" H 5438 1850 50  0001 C CNN
@@
 AR Path="/5D4F34CB/5D58662A" Ref="R?"  Part="1"
 AR Path="/5D167BBA/5D58662A" Ref="R204"  Part="1"
-F 0 "R104" V 5550 1250 50  0000 C CNN
+F 0 "R204" V 5550 1250 50  0000 C CNN
 F 1 "1M" V 5650 1250 50  0000 C CNN
 F 2 "Resistor_SMD:R_0805_2012Metric" V 5580 1250 50  0001 C CNN
@@
 AR Path="/5D4F34CB/5D58663B" Ref="C?"  Part="1"
 AR Path="/5D167BBA/5D58663B" Ref="C203"  Part="1"
-F 0 "C103" H 8615 1196 50  0000 L CNN
+F 0 "C203" H 8615 1196 50  0000 L CNN
 F 1 "1u" H 8615 1105 50  0000 L CNN
 F 2 "Capacitor_SMD:C_0805_2012Metric" H 8538 1000 50  0001 C CNN
@@
 AR Path="/5D4F34CB/5D58664A" Ref="R?"  Part="1"
 AR Path="/5D167BBA/5D58664A" Ref="R205"  Part="1"
-F 0 "R105" V 5550 1450 50  0000 C CNN
+F 0 "R205" V 5550 1450 50  0000 C CNN
 F 1 "1M" V 5650 1450 50  0000 C CNN
 F 2 "Resistor_SMD:R_0805_2012Metric" V 5580 1450 50  0001 C CNN
@@
 AR Path="/5D4F34CB/5D586651" Ref="R?"  Part="1"
 AR Path="/5D167BBA/5D586651" Ref="R206"  Part="1"
-F 0 "R106" V 5550 1650 50  0000 C CNN
+F 0 "R206" V 5550 1650 50  0000 C CNN
 F 1 "1M" V 5650 1650 50  0000 C CNN
 F 2 "Resistor_SMD:R_0805_2012Metric" V 5580 1650 50  0001 C CNN
@@
 AR Path="/5D4F34CB/5D586658" Ref="R?"  Part="1"
 AR Path="/5D167BBA/5D586658" Ref="R207"  Part="1"
-F 0 "R107" V 5550 1850 50  0000 C CNN
+F 0 "R207" V 5550 1850 50  0000 C CNN
 F 1 "1M" V 5650 1850 50  0000 C CNN
 F 2 "Resistor_SMD:R_0805_2012Metric" V 5580 1850 50  0001 C CNN
@@
 AR Path="/5D4F34CB/5D58669D" Ref="R?"  Part="1"
 AR Path="/5D167BBA/5D58669D" Ref="R202"  Part="1"
-F 0 "R102" V 5050 5800 50  0000 C CNN
+F 0 "R202" V 5050 5800 50  0000 C CNN
 F 1 "1k" V 5150 5800 50  0000 C CNN
 F 2 "Resistor_SMD:R_0805_2012Metric" V 5080 5800 50  0001 C CNN
@@
 AR Path="/5D4F34CB/5D5866B2" Ref="R?"  Part="1"
 AR Path="/5D167BBA/5D5866B2" Ref="R208"  Part="1"
-F 0 "R108" V 5550 5800 50  0000 C CNN
+F 0 "R208" V 5550 5800 50  0000 C CNN
 F 1 "1k" V 5650 5800 50  0000 C CNN
 F 2 "Resistor_SMD:R_0805_2012Metric" V 5580 5800 50  0001 C CNN
@@
 AR Path="/5D4F34CB/5D7CA317" Ref="#PWR?"  Part="1"
 AR Path="/5D167BBA/5D7CA317" Ref="#PWR?"  Part="1"
-F 0 "#PWR0106" H 7400 5150 50  0001 C CNN
+F 0 "#PWR?" H 7400 5150 50  0001 C CNN
 F 1 "GND" H 7400 5250 50  0000 C CNN
 F 2 "" H 7400 5400 50  0001 C CNN
